Commit message: formation working, still issues on self_positioning

File: robots/flying_camera.urdf.xacro (robot description, xacro)
@@ -1,4 +1,5 @@
 <?xml version="1.0" encoding="UTF-8"?>
 <robot xmlns:xacro="http://ros.org/wiki/xacro" name="flying_camera">
+    <xacro:arg name="id" default="-1" />
 	<!-- Joints controller -->
 	<xacro:include filename="$(find opt_view)/gazebo/ros_control.urdf" />
@@ -8,5 +9,5 @@
 	<xacro:include filename="$(find rotors_description)/urdf/$(arg mav_name)_base.xacro" />
 	<xacro:camera_joint parent="${namespace}/base_link"
-		prefix="" namespace="${namespace}">
+		prefix="" namespace="">
 		<origin xyz="0 0.0 0" rpy="${pi} 0 0" />
 	</xacro:camera_joint>
@@ -22,5 +23,5 @@
     odometry_topic="uav_odometry/odometry"
     parent_frame_id="world"
-    child_frame_id="uav_odometry4"
+    child_frame_id="$(arg id)"
     mass_odometry_sensor="0.00001"
     measurement_divisor="1"

File: urdf/camera_joint.transmission.xacro (robot description, xacro)
@@ -5,10 +5,10 @@
        xmlns:xacro="http://ros.org/wiki/xacro">
 	<xacro:macro name="widowx_arm_transmission" params="prefix namespace">
-		<transmission name="${namespace}/${prefix}_tran_1">
+		<transmission name="tran_1">
 			<type>transmission_interface/SimpleTransmission</type>
-			<joint name="${namespace}/${prefix}camera_joint">
+			<joint name="camera_joint">
 				<hardwareInterface>hardware_interface/VelocityJointInterface</hardwareInterface>
 			</joint>
-			<actuator name="${namespace}/${prefix)_motor1">
+			<actuator name="motor1">
 				<hardwareInterface>hardware_interface/VelocityJointInterface</hardwareInterface>
 				<mechanicalReduction>1</mechanicalReduction>

File: urdf/camera_joint.urdf.xacro (robot description, xacro)
@@ -4,9 +4,9 @@
 	<xacro:macro name="camera_joint" params="parent namespace prefix *origin">
 		<!-- Links -->
-		<link name="${namespace}/${prefix}camera_base_link" parent="${parent}">
+		<link name="camera_base_link" parent="${parent}">
 			<collision>
 				<origin xyz="0 0 0" rpy="0 0 0" />
 				<geometry>
-					<box size="0.05 0.05 0.05" />
+					<box size="0.0005 0.0005 0.0005" />
 				</geometry>
 			</collision>
@@ -14,5 +14,5 @@
 				<origin xyz="0 0 0" rpy="0 0 0" />
 				<geometry>
-					<box size="0.05 0.05 0.05" />
+					<box size="0.0005 0.0005 0.0005" />
 				</geometry>
 			</visual>
@@ -23,10 +23,10 @@
 			</inertial>
 		</link>
-		<link name="${namespace}/${prefix}camera_link"
-			parent="${namespace}/${prefix}camera_base_link">
+		<link name="camera_link"
+			parent="camera_base_link">
 			<visual>
-				<origin  xyz="0 0 0" rpy="0 0 0" />
+				<origin  xyz="0 0 0.01" rpy="0 0 0" />
 				<geometry>
-					<mesh filename="package://opt_view/meshes/camera.dae" />
+					<mesh filename="package://opt_view/meshes/camera.dae" scale="0.5 0.5 0.5"/>
 				</geometry>
 			</visual>
@@ -34,5 +34,5 @@
 				<origin xyz="0 0 0" rpy="0 0 0" />
 				<geometry>
-					<box size="0.05 0.05 0.05" />
+					<box size="0.0005 0.0005 0.0005" />
 				</geometry>
 			</collision>
@@ -43,17 +43,80 @@
 			</inertial>
 		</link>
+		<link name="camera_plugin_link">
+			<visual>
+				<origin  xyz="0 0 0.01" rpy="0 0 0" />
+				<geometry>
+					<box size="0.0005 0.0005 0.0005" />
+				</geometry>
+			</visual>
+			<collision>
+				<origin xyz="0 0 0" rpy="0 0 0" />
+				<geometry>
+					<box size="0.0 0.00 0.000" />
+				</geometry>
+			</collision>
+			<inertial>
+				<origin xyz="0 0 0" rpy="0 0 0" />
+				<mass value="0.0001" />
+				<inertia ixx="0.00002" ixy="0.0" ixz="0.0" iyy="0.00002" iyz="0.0" izz="0.00002" />
+			</inertial>
+		</link>
 		<!-- Joints -->
-		<joint name="${namespace}/${prefix}camera_base_joint" type="fixed">
+		<joint name="camera_base_joint" type="fixed">
 			<xacro:insert_block name="origin" />
 			<parent link="${parent}" />
-			<child link="${namespace}/${prefix}camera_base_link"/>
+			<child link="camera_base_link"/>
 		</joint>
-		<joint name="${namespace}/${prefix}camera_joint" type="revolute">
+		<joint name="camera_joint" type="revolute">
 			<origin xyz="0 0 0" rpy="0 0 0" />
-			<parent link="${namespace}/${prefix}camera_base_link" />
-			<child link="${namespace}/${prefix}camera_link" />
+			<parent link="camera_base_link" />
+			<child link="camera_link" />
 			<axis xyz="0 0 1" />
 			<limit lower="${-pi/2}" upper="${pi/2}" velocity="100" effort="100" />
 		</joint>
+		<joint name="camera_plugin_joint" type="fixed">
+			<origin xyz="0.05 0 0.1" rpy="${pi} ${-pi/4} 0" />
+			<parent link="camera_link" />
+			<child link="camera_plugin_link" />
+		</joint>
+		<gazebo reference="camera_plugin_link">
+			<sensor type="camera" name="camera1">
+				<update_rate>30.0</update_rate>
+				<camera name="head">
+					<horizontal_fov>1.3962634</horizontal_fov>
+					<image>
+						<width>800</width>
+						<height>800</height>
+						<format>R8G8B8</format>
+					</image>
+					<clip>
+						<near>0.02</near>
+						<far>300</far>
+					</clip>
+					<noise>
+						<type>gaussian</type>
+						<!-- Noise is sampled independently per pixel on each frame.
+						That pixel's noise value is added to each of its color
+						channels, which at that point lie in the range [0,1]. -->
+						<mean>0.0</mean>
+						<stddev>0.007</stddev>
+					</noise>
+				</camera>
+				<plugin name="camera_controller" filename="libgazebo_ros_camera.so">
+					<alwaysOn>true</alwaysOn>
+					<updateRate>0.0</updateRate>
+					<cameraName>camera1</cameraName>
+					<imageTopicName>image_raw</imageTopicName>
+					<cameraInfoTopicName>camera_info</cameraInfoTopicName>
+					<frameName>camera_link</frameName>
+					<hackBaseline>0.07</hackBaseline>
+					<distortionK1>0.0</distortionK1>
+					<distortionK2>0.0</distortionK2>
+					<distortionK3>0.0</distortionK3>
+					<distortionT1>0.0</distortionT1>
+					<distortionT2>0.0</distortionT2>
+				</plugin>
+			</sensor>
+		</gazebo>
 		<xacro:widowx_arm_transmission prefix="${prefix}" namespace="${namespace}" />
 	</xacro:macro>

Commit message: multiple views - started backprojection

File: robots/flying_camera.urdf.xacro (robot description, xacro)
@@ -42,3 +42,38 @@
     <origin xyz="0.0 0.0 0.0" rpy="0.0 0.0 0.0" />
   </xacro:odometry_plugin_macro>
+  <xacro:odometry_plugin_macro
+    namespace="${namespace}"
+    odometry_sensor_suffix="5"
+    parent_link="camera_plugin_link"
+    pose_topic="camera_odometry/pose"
+    pose_with_covariance_topic="camera_odometry/pose_with_covariance"
+    position_topic="camera_odometry/position"
+    transform_topic="camera_odometry/transform"
+    odometry_topic="camera_odometry/odometry"
+    parent_frame_id="world"
+    child_frame_id="$(arg id)"
+    mass_odometry_sensor="0.00001"
+    measurement_divisor="1"
+    measurement_delay="0"
+    unknown_delay="0.0"
+    noise_normal_position="0 0 0"
+    noise_normal_quaternion="0 0 0"
+    noise_normal_linear_velocity="0 0 0"
+    noise_normal_angular_velocity="0 0 0"
+    noise_uniform_position="0 0 0"
+    noise_uniform_quaternion="0 0 0"
+    noise_uniform_linear_velocity="0 0 0"
+    noise_uniform_angular_velocity="0 0 0"
+    enable_odometry_map="false"
+    odometry_map=""
+    image_scale="">
+    <inertia ixx="0.00001" ixy="0.0" ixz="0.0" iyy="0.00001" iyz="0.0" izz="0.00001" /> <!-- [kg m^2] [kg m^2] [kg m^2] [kg m^2] [kg m^2] [kg m^2] -->
+    <origin xyz="0.0 0.0 0.0" rpy="0.0 0.0 0.0" />
+  </xacro:odometry_plugin_macro>
+  <gazebo>
+    <plugin name="visibility_grid_plugin" filename="libvisibility_grid.so">
+      <camera_odom_topic>/uavs/agent_$(arg id)/camera_odometry/odometry</camera_odom_topic>
+      <projected_view_topic>/uavs/agent_$(arg id)/predicted_view/update</projected_view_topic>
+    </plugin>
+  </gazebo>
 </robot>

Commit message: temp checkout

File: robots/flying_camera.urdf.xacro (robot description, xacro)
@@ -71,5 +71,5 @@
     <origin xyz="0.0 0.0 0.0" rpy="0.0 0.0 0.0" />
   </xacro:odometry_plugin_macro>
-  <gazebo>
+  <gazebo reference="camera_plugin_visual">
     <plugin name="visibility_grid_plugin" filename="libvisibility_grid.so">
       <camera_odom_topic>/uavs/agent_$(arg id)/camera_odometry/odometry</camera_odom_topic>

File: urdf/camera_joint.urdf.xacro (robot description, xacro)
@@ -44,5 +44,5 @@
 		</link>
 		<link name="camera_plugin_link">
-			<visual>
+			<visual name="camera_plugin_visual">
 				<origin  xyz="0 0 0.01" rpy="0 0 0" />
 				<geometry>

Commit message: non funziona visual

File: robots/flying_camera.urdf.xacro (robot description, xacro)
@@ -9,5 +9,5 @@
 	<xacro:include filename="$(find rotors_description)/urdf/$(arg mav_name)_base.xacro" />
 	<xacro:camera_joint parent="${namespace}/base_link"
-		prefix="" namespace="">
+		prefix="" namespace="" id="$(arg id)">
 		<origin xyz="0 0.0 0" rpy="${pi} 0 0" />
 	</xacro:camera_joint>
@@ -68,13 +68,6 @@
     odometry_map=""
     image_scale="">
-    <inertia ixx="0.00001" ixy="0.0" ixz="0.0" iyy="0.00001" iyz="0.0" izz="0.00001" /> <!-- [kg m^2] [kg m^2] [kg m^2] [kg m^2] [kg m^2] [kg m^2] -->
+    <inertia ixx="0.00001" ixy="0.0" ixz="0.0" iyy="0.00001" iyz="0.0" izz="0.00001" />
     <origin xyz="0.0 0.0 0.0" rpy="0.0 0.0 0.0" />
   </xacro:odometry_plugin_macro>
-  <gazebo reference="camera_plugin_visual">
-    <plugin name="visibility_grid_plugin" filename="libvisibility_grid.so">
-      <camera_odom_topic>/uavs/agent_$(arg id)/camera_odometry/odometry</camera_odom_topic>
-      <projected_view_topic>/uavs/agent_$(arg id)/predicted_view/update</projected_view_topic>
-      <id>$(arg id)</id>
-    </plugin>
-  </gazebo>
 </robot>

File: urdf/camera_joint.urdf.xacro (robot description, xacro)
@@ -2,5 +2,5 @@
 <robot xmlns:xacro="http://ros.org/wiki/xacro">
 	<xacro:include filename="$(find opt_view)/urdf/camera_joint.transmission.xacro" />
-	<xacro:macro name="camera_joint" params="parent namespace prefix *origin">
+	<xacro:macro name="camera_joint" params="parent namespace prefix id *origin">
 		<!-- Links -->
 		<link name="camera_base_link" parent="${parent}">
@@ -44,20 +44,8 @@
 		</link>
 		<link name="camera_plugin_link">
-			<visual name="camera_plugin_visual">
-				<origin  xyz="0 0 0.01" rpy="0 0 0" />
-				<geometry>
-					<box size="0.0005 0.0005 0.0005" />
-				</geometry>
-			</visual>
-			<collision>
-				<origin xyz="0 0 0" rpy="0 0 0" />
-				<geometry>
-					<box size="0.0 0.00 0.000" />
-				</geometry>
-			</collision>
 			<inertial>
 				<origin xyz="0 0 0" rpy="0 0 0" />
-				<mass value="0.0001" />
-				<inertia ixx="0.00002" ixy="0.0" ixz="0.0" iyy="0.00002" iyz="0.0" izz="0.00002" />
+				<mass value="0.01" />
+				<inertia ixx="0.002" ixy="0.0" ixz="0.0" iyy="0.002" iyz="0.0" izz="0.002" />
 			</inertial>
 		</link>
