Commit message: projected visual funzionante

File: urdf/camera_joint.urdf.xacro (robot description, xacro)
@@ -64,5 +64,5 @@
 		</joint>
 		<joint name="camera_plugin_joint" type="fixed">
-			<origin xyz="0.05 0 0.1" rpy="${pi} ${-pi/4} 0" />
+			<origin xyz="0.05 0 0.1" rpy="${pi} ${-pi/3} 0" />
 			<parent link="camera_link" />
 			<child link="camera_plugin_link" />

Commit message: opt

File: urdf/camera_joint.urdf.xacro (robot description, xacro)
@@ -2,11 +2,11 @@
 <robot xmlns:xacro="http://ros.org/wiki/xacro">
 	<xacro:include filename="$(find opt_view)/urdf/camera_joint.transmission.xacro" />
-	<xacro:macro name="camera_joint" params="parent namespace prefix id *origin">
+	<xacro:macro name="camera_joint" params="parent namespace prefix *origin">
 		<!-- Links -->
-		<link name="camera_base_link" parent="${parent}">
+		<link name="${namespace}/${prefix}camera_base_link" parent="${parent}">
 			<collision>
 				<origin xyz="0 0 0" rpy="0 0 0" />
 				<geometry>
-					<box size="0.0005 0.0005 0.0005" />
+					<box size="0.05 0.05 0.05" />
 				</geometry>
 			</collision>
@@ -14,5 +14,5 @@
 				<origin xyz="0 0 0" rpy="0 0 0" />
 				<geometry>
-					<box size="0.0005 0.0005 0.0005" />
+					<box size="0.05 0.05 0.05" />
 				</geometry>
 			</visual>
@@ -23,10 +23,10 @@
 			</inertial>
 		</link>
-		<link name="camera_link"
-			parent="camera_base_link">
+		<link name="${namespace}/${prefix}camera_link"
+			parent="${namespace}/${prefix}camera_base_link">
 			<visual>
-				<origin  xyz="0 0 0.01" rpy="0 0 0" />
+				<origin  xyz="0 0 0" rpy="0 0 0" />
 				<geometry>
-					<mesh filename="package://opt_view/meshes/camera.dae" scale="0.5 0.5 0.5"/>
+					<mesh filename="package://opt_view/meshes/camera.dae" />
 				</geometry>
 			</visual>
@@ -34,5 +34,5 @@
 				<origin xyz="0 0 0" rpy="0 0 0" />
 				<geometry>
-					<box size="0.0005 0.0005 0.0005" />
+					<box size="0.05 0.05 0.05" />
 				</geometry>
 			</collision>
@@ -43,68 +43,17 @@
 			</inertial>
 		</link>
-		<link name="camera_plugin_link">
-			<inertial>
-				<origin xyz="0 0 0" rpy="0 0 0" />
-				<mass value="0.01" />
-				<inertia ixx="0.002" ixy="0.0" ixz="0.0" iyy="0.002" iyz="0.0" izz="0.002" />
-			</inertial>
-		</link>
 		<!-- Joints -->
-		<joint name="camera_base_joint" type="fixed">
+		<joint name="${namespace}/${prefix}camera_base_joint" type="fixed">
 			<xacro:insert_block name="origin" />
 			<parent link="${parent}" />
-			<child link="camera_base_link"/>
+			<child link="${namespace}/${prefix}camera_base_link"/>
 		</joint>
-		<joint name="camera_joint" type="revolute">
+		<joint name="${namespace}/${prefix}camera_joint" type="revolute">
 			<origin xyz="0 0 0" rpy="0 0 0" />
-			<parent link="camera_base_link" />
-			<child link="camera_link" />
+			<parent link="${namespace}/${prefix}camera_base_link" />
+			<child link="${namespace}/${prefix}camera_link" />
 			<axis xyz="0 0 1" />
 			<limit lower="${-pi/2}" upper="${pi/2}" velocity="100" effort="100" />
 		</joint>
-		<joint name="camera_plugin_joint" type="fixed">
-			<origin xyz="0.05 0 0.1" rpy="${pi} ${-pi/3} 0" />
-			<parent link="camera_link" />
-			<child link="camera_plugin_link" />
-		</joint>
-		<gazebo reference="camera_plugin_link">
-			<sensor type="camera" name="camera1">
-				<update_rate>30.0</update_rate>
-				<camera name="head">
-					<horizontal_fov>1.3962634</horizontal_fov>
-					<image>
-						<width>800</width>
-						<height>800</height>
-						<format>R8G8B8</format>
-					</image>
-					<clip>
-						<near>0.02</near>
-						<far>300</far>
-					</clip>
-					<noise>
-						<type>gaussian</type>
-						<!-- Noise is sampled independently per pixel on each frame.
-						That pixel's noise value is added to each of its color
-						channels, which at that point lie in the range [0,1]. -->
-						<mean>0.0</mean>
-						<stddev>0.007</stddev>
-					</noise>
-				</camera>
-				<plugin name="camera_controller" filename="libgazebo_ros_camera.so">
-					<alwaysOn>true</alwaysOn>
-					<updateRate>0.0</updateRate>
-					<cameraName>camera1</cameraName>
-					<imageTopicName>image_raw</imageTopicName>
-					<cameraInfoTopicName>camera_info</cameraInfoTopicName>
-					<frameName>camera_link</frameName>
-					<hackBaseline>0.07</hackBaseline>
-					<distortionK1>0.0</distortionK1>
-					<distortionK2>0.0</distortionK2>
-					<distortionK3>0.0</distortionK3>
-					<distortionT1>0.0</distortionT1>
-					<distortionT2>0.0</distortionT2>
-				</plugin>
-			</sensor>
-		</gazebo>
 		<xacro:widowx_arm_transmission prefix="${prefix}" namespace="${namespace}" />
 	</xacro:macro>

Commit message: loss probability inclusa nell'ottimizzazione - funziona - progetto finito

File: urdf/camera_joint.urdf.xacro (robot description, xacro)
@@ -2,11 +2,11 @@
 <robot xmlns:xacro="http://ros.org/wiki/xacro">
 	<xacro:include filename="$(find opt_view)/urdf/camera_joint.transmission.xacro" />
-	<xacro:macro name="camera_joint" params="parent namespace prefix *origin">
+	<xacro:macro name="camera_joint" params="parent namespace prefix id *origin">
 		<!-- Links -->
-		<link name="${namespace}/${prefix}camera_base_link" parent="${parent}">
+		<link name="camera_base_link" parent="${parent}">
 			<collision>
 				<origin xyz="0 0 0" rpy="0 0 0" />
 				<geometry>
-					<box size="0.05 0.05 0.05" />
+					<box size="0.0005 0.0005 0.0005" />
 				</geometry>
 			</collision>
@@ -14,5 +14,5 @@
 				<origin xyz="0 0 0" rpy="0 0 0" />
 				<geometry>
-					<box size="0.05 0.05 0.05" />
+					<box size="0.0005 0.0005 0.0005" />
 				</geometry>
 			</visual>
@@ -23,10 +23,10 @@
 			</inertial>
 		</link>
-		<link name="${namespace}/${prefix}camera_link"
-			parent="${namespace}/${prefix}camera_base_link">
+		<link name="camera_link"
+			parent="camera_base_link">
 			<visual>
-				<origin  xyz="0 0 0" rpy="0 0 0" />
+				<origin  xyz="0 0 0.01" rpy="0 0 0" />
 				<geometry>
-					<mesh filename="package://opt_view/meshes/camera.dae" />
+					<mesh filename="package://opt_view/meshes/camera.dae" scale="0.5 0.5 0.5"/>
 				</geometry>
 			</visual>
@@ -34,5 +34,5 @@
 				<origin xyz="0 0 0" rpy="0 0 0" />
 				<geometry>
-					<box size="0.05 0.05 0.05" />
+					<box size="0.0005 0.0005 0.0005" />
 				</geometry>
 			</collision>
@@ -43,17 +43,68 @@
 			</inertial>
 		</link>
+		<link name="camera_plugin_link">
+			<inertial>
+				<origin xyz="0 0 0" rpy="0 0 0" />
+				<mass value="0.01" />
+				<inertia ixx="0.002" ixy="0.0" ixz="0.0" iyy="0.002" iyz="0.0" izz="0.002" />
+			</inertial>
+		</link>
 		<!-- Joints -->
-		<joint name="${namespace}/${prefix}camera_base_joint" type="fixed">
+		<joint name="camera_base_joint" type="fixed">
 			<xacro:insert_block name="origin" />
 			<parent link="${parent}" />
-			<child link="${namespace}/${prefix}camera_base_link"/>
+			<child link="camera_base_link"/>
 		</joint>
-		<joint name="${namespace}/${prefix}camera_joint" type="revolute">
+		<joint name="camera_joint" type="revolute">
 			<origin xyz="0 0 0" rpy="0 0 0" />
-			<parent link="${namespace}/${prefix}camera_base_link" />
-			<child link="${namespace}/${prefix}camera_link" />
+			<parent link="camera_base_link" />
+			<child link="camera_link" />
 			<axis xyz="0 0 1" />
 			<limit lower="${-pi/2}" upper="${pi/2}" velocity="100" effort="100" />
 		</joint>
+		<joint name="camera_plugin_joint" type="fixed">
+			<origin xyz="0.05 0 0.1" rpy="${pi} ${-pi/3} 0" />
+			<parent link="camera_link" />
+			<child link="camera_plugin_link" />
+		</joint>
+		<gazebo reference="camera_plugin_link">
+			<sensor type="camera" name="camera1">
+				<update_rate>30.0</update_rate>
+				<camera name="head">
+					<horizontal_fov>1.3962634</horizontal_fov>
+					<image>
+						<width>800</width>
+						<height>800</height>
+						<format>R8G8B8</format>
+					</image>
+					<clip>
+						<near>0.02</near>
+						<far>300</far>
+					</clip>
+					<noise>
+						<type>gaussian</type>
+						<!-- Noise is sampled independently per pixel on each frame.
+						That pixel's noise value is added to each of its color
+						channels, which at that point lie in the range [0,1]. -->
+						<mean>0.0</mean>
+						<stddev>0.007</stddev>
+					</noise>
+				</camera>
+				<plugin name="camera_controller" filename="libgazebo_ros_camera.so">
+					<alwaysOn>true</alwaysOn>
+					<updateRate>0.0</updateRate>
+					<cameraName>camera1</cameraName>
+					<imageTopicName>image_raw</imageTopicName>
+					<cameraInfoTopicName>camera_info</cameraInfoTopicName>
+					<frameName>camera_link</frameName>
+					<hackBaseline>0.07</hackBaseline>
+					<distortionK1>0.0</distortionK1>
+					<distortionK2>0.0</distortionK2>
+					<distortionK3>0.0</distortionK3>
+					<distortionT1>0.0</distortionT1>
+					<distortionT2>0.0</distortionT2>
+				</plugin>
+			</sensor>
+		</gazebo>
 		<xacro:widowx_arm_transmission prefix="${prefix}" namespace="${namespace}" />
 	</xacro:macro>

Commit message: params evasion3.mp4

File: urdf/camera_joint.urdf.xacro (robot description, xacro)
@@ -57,5 +57,5 @@
 		</joint>
 		<joint name="camera_joint" type="revolute">
-			<origin xyz="0 0 0" rpy="0 0 0" />
+			<origin xyz="-0.02 -0.035 0" rpy="0 0 0" />
 			<parent link="camera_base_link" />
 			<child link="camera_link" />
